Commit message: lidar done in gazebo topic not visible for some reason - WIP

File: mir100/mir.urdf.xacro (robot description, xacro)
@@ -17,4 +17,5 @@
   <!-- Custom camera -->
   <xacro:include filename="$(find ai3-roai-project)/mir100/camera.urdf.xacro" />
+  <xacro:include filename="$(find ai3-roai-project)/mir100/lidar.urdf.xacro" />
   <!-- instead of the controller_plugin_gazebo, you can use the diffdrive controller like this:
     <xacro:diff_controller_plugin_gazebo prefix=""
@@ -24,3 +25,7 @@
       wheel_radius="${mir_act_wheel_radius}"/>
   -->
+  <!-- <xacro:include filename="inertial_macros.xacro"/> -->
+  <material name="red">
+    <color rgba="1 0 0 1"/>
+  </material>
 </robot>
