Commit message: fixed lidar to publish data to /scan

File: mir100/lidar.urdf.xacro (robot description, xacro)
@@ -3,5 +3,4 @@
     <xacro:include filename="inertial_macros.xacro"/>
     <joint name="laser_joint" type="fixed">
-        <!-- <parent link="chassis"/> -->
         <parent link="base_link" />
         <child link="laser_frame"/>
@@ -43,10 +42,7 @@
                 </range>
             </ray>
-            <plugin name="laser_controller" filename="libgazebo_ros_ray_sensor.so">
-                <ros>
-                    <argument>~/out:=scan</argument>
-                </ros>
-                <output_type>sensor_msgs/LaserScan</output_type>
-                <frame_name>laser_frame</frame_name>
+            <plugin name="laser_controller" filename="libgazebo_ros_gpu_laser.so">
+                <topicName>/scan</topicName>
+                <frameName>laser_frame</frameName>
             </plugin>
         </sensor>

Commit message: adjusted lidar link naming

File: mir100/lidar.urdf.xacro (robot description, xacro)
@@ -4,8 +4,8 @@
     <joint name="laser_joint" type="fixed">
         <parent link="base_link" />
-        <child link="laser_frame"/>
+        <child link="base_laser_link"/>
         <origin xyz="0.1 0 0.4" rpy="0 0 1.5708"/>
     </joint>
-    <link name="laser_frame">
+    <link name="base_laser_link">
         <visual>
             <geometry>
@@ -23,5 +23,5 @@
         </xacro:inertial_cylinder>
     </link>
-    <gazebo reference="laser_frame">
+    <gazebo reference="base_laser_link">
         <material>Gazebo/Red</material>
         <sensor name="laser" type="ray">
@@ -44,5 +44,5 @@
             <plugin name="laser_controller" filename="libgazebo_ros_gpu_laser.so">
                 <topicName>/scan</topicName>
-                <frameName>laser_frame</frameName>
+                <frameName>base_laser_link</frameName>
             </plugin>
         </sensor>

Commit message: extended laser range

File: mir100/lidar.urdf.xacro (robot description, xacro)
@@ -1,24 +1,24 @@
 <?xml version="1.0"?>
-<robot xmlns:xacro="http://www.ros.org/wiki/xacro" >
-    <xacro:include filename="inertial_macros.xacro"/>
+<robot xmlns:xacro="http://www.ros.org/wiki/xacro">
+    <xacro:include filename="inertial_macros.xacro" />
     <joint name="laser_joint" type="fixed">
         <parent link="base_link" />
-        <child link="base_laser_link"/>
-        <origin xyz="0.1 0 0.4" rpy="0 0 1.5708"/>
+        <child link="base_laser_link" />
+        <origin xyz="0.1 0 0.4" rpy="0 0 1.5708" />
     </joint>
     <link name="base_laser_link">
         <visual>
             <geometry>
-                <cylinder radius="0.05" length="0.04"/>
+                <cylinder radius="0.05" length="0.04" />
             </geometry>
-            <material name="red"/>
+            <material name="red" />
         </visual>
         <collision>
             <geometry>
-                <cylinder radius="0.05" length="0.04"/>
+                <cylinder radius="0.05" length="0.04" />
             </geometry>
         </collision>
         <xacro:inertial_cylinder mass="0.1" length="0.04" radius="0.05">
-            <origin xyz="0 0 0" rpy="0 0 0"/>
+            <origin xyz="0 0 0" rpy="0 0 0" />
         </xacro:inertial_cylinder>
     </link>
@@ -39,5 +39,5 @@
                 <range>
                     <min>0.3</min>
-                    <max>12</max>
+                    <max>100</max>
                 </range>
             </ray>
